File: fingerprint/fingerprint.kicad_sch (KiCad schematic)
At the start: 11 parts

Commit message: up
Parts:
- added Electromagnetic: Lock, Inductor_SMD:L_6.3x6.3_H3, symbol Device:LED
Connections:
- net INPUT3: now reaches A1.17 (D2)
- net INPUT2: now reaches A1.18 (D3)
- net NO: no longer names the net of Relay.14
- net NO: now also Electromagnetic.2 (A)
- new net GND2: Electromagnetic.1 (K)
Changed lines of the file:
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@@
-    (stroke (width 0) (type default))
-  )
-  (wire (pts (xy 243.84 34.29) (xy 243.84 33.02))
     (stroke (width 0) (type default))
   )
@@
     (stroke (width 0) (type default))
   )
+  (wire (pts (xy 243.84 33.02) (xy 262.89 33.02))
+    (stroke (width 0) (type default))
+  )
   (wire (pts (xy 241.3 52.07) (xy 241.3 49.53))
     (stroke (width 0) (type default))
   )
+  (wire (pts (xy 243.84 33.02) (xy 243.84 34.29))
+    (stroke (width 0) (type default))
+  )
+  (wire (pts (xy 238.76 29.21) (xy 238.76 34.29))
+    (stroke (width 0) (type default))
+  )
   (wire (pts (xy 205.74 41.91) (xy 205.74 48.26))
     (stroke (width 0) (type default))
@@
     (stroke (width 0) (type default))
   )
-  (wire (pts (xy 238.76 34.29) (xy 238.76 29.21))
-    (stroke (width 0) (type default))
-  )
   (wire (pts (xy 214.63 34.29) (xy 214.63 40.64))
     (stroke (width 0) (type default))
   )
-  (wire (pts (xy 243.84 33.02) (xy 248.92 33.02))
+  (wire (pts (xy 262.89 38.1) (xy 262.89 33.02))
     (stroke (width 0) (type default))
   )
@@
     (stroke (width 0) (type default))
   )
+  (wire (pts (xy 66.04 68.58) (xy 74.93 68.58))
+    (stroke (width 0) (type default))
+  )
   (wire (pts (xy 214.63 34.29) (xy 231.14 34.29))
     (stroke (width 0) (type default))
   )
+  (wire (pts (xy 262.89 45.72) (xy 262.89 50.8))
+    (stroke (width 0) (type default))
+  )
   (wire (pts (xy 218.44 67.31) (xy 223.52 67.31))
     (stroke (width 0) (type default))
   )
+  (wire (pts (xy 66.04 66.04) (xy 74.93 66.04))
+    (stroke (width 0) (type default))
+  )
   (wire (pts (xy 66.04 55.88) (xy 74.93 55.88))
     (stroke (width 0) (type default))
@@
     (effects (font (size 1.27 1.27)) (justify left bottom))
   )
+  (label "INPUT2" (at 68.58 66.04 0) (fields_autoplaced)
+    (effects (font (size 1.27 1.27)) (justify left bottom))
+  )
+  (label "INPUT3" (at 68.58 68.58 0) (fields_autoplaced)
+    (effects (font (size 1.27 1.27)) (justify left bottom))
+  )
   (label "NC" (at 248.92 29.21 0) (fields_autoplaced)
     (effects (font (size 1.27 1.27)) (justify left bottom))
   )
-  (label "NO" (at 248.92 33.02 0) (fields_autoplaced)
+  (label "NO - 12V lock" (at 242.57 33.02 0) (fields_autoplaced)
     (effects (font (size 1.27 1.27)) (justify left bottom))
   )
@@
     )
   )
+  (symbol (lib_id "Device:LED") (at 262.89 41.91 90) (unit 1)
+    (in_bom yes) (on_board yes) (dnp no) (fields_autoplaced)
+    (property "Reference" "Electromagnetic" (at 266.7 42.8625 90)
+      (effects (font (size 1.27 1.27)) (justify right))
+    )
+    (property "Value" "Lock" (at 266.7 45.4025 90)
+      (effects (font (size 1.27 1.27)) (justify right))
+    )
+    (property "Footprint" "Inductor_SMD:L_6.3x6.3_H3" (at 262.89 41.91 0)
+      (effects (font (size 1.27 1.27)) hide)
+    )
+    (property "Datasheet" "~" (at 262.89 41.91 0)
+      (effects (font (size 1.27 1.27)) hide)
+    )
+    (pin "1")
+    (pin "2")
+    (instances
+      (project "fingerprint"
+        (path "/c6978c6a-d0b0-48b8-9e51-442c42e84720"
+          (reference "Electromagnetic") (unit 1)
+        )
+      )
+    )
+  )
   (symbol (lib_id "Device:LED") (at 205.74 52.07 90) (unit 1)
     (in_bom yes) (on_board yes) (dnp no) (fields_autoplaced)
@@
         )
       )
+    )
+  )
+  (symbol (lib_id "power:GND2") (at 262.89 50.8 0) (unit 1)
+    (in_bom yes) (on_board yes) (dnp no) (fields_autoplaced)
+    (property "Reference" "#PWR05" (at 262.89 57.15 0)
+      (effects (font (size 1.27 1.27)) hide)
+    )
+    (property "Value" "GND2" (at 262.89 55.88 0)
+      (effects (font (size 1.27 1.27)))
+    )
+    (property "Footprint" "" (at 262.89 50.8 0)
+      (effects (font (size 1.27 1.27)) hide)
+    )
+    (property "Datasheet" "" (at 262.89 50.8 0)
+      (effects (font (size 1.27 1.27)) hide)
+    )
+    (pin "1")
+    (instances
+      (project "fingerprint"
+        (path "/c6978c6a-d0b0-48b8-9e51-442c42e84720"
+          (reference "#PWR05") (unit 1)
+        )
+      )
